File: Nano SwinSIDb.sch (KiCad schematic (older format))
At the start: 18 parts, among them J5 6PinConnector, U1 ATmega88PA-AU, U2 6581 Pins, U3 6581 Socket, X1 ECS-3225MV

Commit message: Completed pcb design and gerber files for manufacture.
Parts:
- U2, U3: symbol 65xx:6581 -> Nano-SwinSIDb-rescue:6581-65xx
Changed lines of the file:
@@
 $EndComp
 $Comp
-L 65xx:6581 U3
+L Nano-SwinSIDb-rescue:6581-65xx U3
 U 1 1 605850ED
 P 2700 5850
@@
 CAP1A
 $Comp
-L 65xx:6581 U2
+L Nano-SwinSIDb-rescue:6581-65xx U2
 U 1 1 605EBB1B
 P 1800 2650
